File: pcb/buffer.brd (EAGLE design)
At the start: 98 x 22 mm, 16 parts, among them IC1 LF353D, IC2 LF353D, IC3 LF353D

Commit message: fix for bad routing
Routing:
- net GND: track 5.57 -> 0.90 mm
Changed lines of the file:
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@@
 </polygon>
 <wire x1="7" y1="11.3" x2="7.9" y2="11.3" width="0.254" layer="1"/>
-<wire x1="7.9" y1="11.3" x2="11.2" y2="8" width="0.254" layer="1"/>
 <polygon width="0.254" layer="1">
 <vertex x="1" y="21"/>
